Commit message: added freshly generated urdfs built from the updated xacros

File: python/rrc_simulation/robot_properties_fingers/urdf/pro/fingerpro.urdf (robot description, URDF)
Before this commit: robot fingerpro, 6 links, 5 joints
Links:
- link finger_lower_link: mass 0.01 -> 0.021
- link finger_middle_link: mass 0.2 -> 0.25
- link finger_tip_link: mass 0.02 -> 0.031
- link finger_upper_link: mass 0.2 -> 0.26

File: python/rrc_simulation/robot_properties_fingers/urdf/pro/trifingerpro.urdf (robot description, URDF)
Before this commit: robot trifingerpro, 17 links, 16 joints
Links:
- link finger_lower_link_0: mass 0.01 -> 0.021
- link finger_lower_link_120: mass 0.01 -> 0.021
- link finger_lower_link_240: mass 0.01 -> 0.021
- link finger_middle_link_0: mass 0.2 -> 0.25
- link finger_middle_link_120: mass 0.2 -> 0.25
- link finger_middle_link_240: mass 0.2 -> 0.25
- link finger_tip_link_0: mass 0.02 -> 0.031
- link finger_tip_link_120: mass 0.02 -> 0.031
- link finger_tip_link_240: mass 0.02 -> 0.031
- link finger_upper_link_0: mass 0.2 -> 0.26
- link finger_upper_link_120: mass 0.2 -> 0.26
- link finger_upper_link_240: mass 0.2 -> 0.26

File: python/rrc_simulation/robot_properties_fingers/urdf/pro/trifingerpro_with_stage.urdf (robot description, URDF)
Before this commit: robot trifingerpro_with_stage, 19 links, 18 joints
Links:
- link finger_lower_link_0: mass 0.01 -> 0.021
- link finger_lower_link_120: mass 0.01 -> 0.021
- link finger_lower_link_240: mass 0.01 -> 0.021
- link finger_middle_link_0: mass 0.2 -> 0.25
- link finger_middle_link_120: mass 0.2 -> 0.25
- link finger_middle_link_240: mass 0.2 -> 0.25
- link finger_tip_link_0: mass 0.02 -> 0.031
- link finger_tip_link_120: mass 0.02 -> 0.031
- link finger_tip_link_240: mass 0.02 -> 0.031
- link finger_upper_link_0: mass 0.2 -> 0.26
- link finger_upper_link_120: mass 0.2 -> 0.26
- link finger_upper_link_240: mass 0.2 -> 0.26

Commit message: fix for tip forces
using split meshes for the tip link (lower + actual tip),
using the contact forces returned by getContactPoints

File: python/rrc_simulation/robot_properties_fingers/urdf/pro/fingerpro.urdf (robot description, URDF)
Before this commit: robot fingerpro, 6 links, 5 joints
Links:
- link finger_tip_link: geometry collision mesh filename=package://robot_properties_fingers/meshes/stl/pro/SIM__BL-F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 scale=1.0 1.0 1.0; visual mesh filename=package://robot_properties_fingers/meshes/stl/pro/SIM__BL-F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 scale=1.0 1.0 1.0

File: python/rrc_simulation/robot_properties_fingers/urdf/pro/trifingerpro.urdf (robot description, URDF)
Before this commit: robot trifingerpro, 17 links, 16 joints
Links:
- link finger_tip_link_0: geometry collision mesh filename=package://robot_properties_fingers/meshes/stl/pro/SIM__BL-F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 scale=1.0 1.0 1.0; visual mesh filename=package://robot_properties_fingers/meshes/stl/pro/SIM__BL-F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 scale=1.0 1.0 1.0
- link finger_tip_link_120: geometry collision mesh filename=package://robot_properties_fingers/meshes/stl/pro/SIM__BL-F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 scale=1.0 1.0 1.0; visual mesh filename=package://robot_properties_fingers/meshes/stl/pro/SIM__BL-F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 scale=1.0 1.0 1.0
- link finger_tip_link_240: geometry collision mesh filename=package://robot_properties_fingers/meshes/stl/pro/SIM__BL-F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 scale=1.0 1.0 1.0; visual mesh filename=package://robot_properties_fingers/meshes/stl/pro/SIM__BL-F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 scale=1.0 1.0 1.0

File: python/rrc_simulation/robot_properties_fingers/urdf/pro/trifingerpro_with_stage.urdf (robot description, URDF)
Before this commit: robot trifingerpro_with_stage, 19 links, 18 joints
Links:
- link finger_tip_link_0: geometry collision mesh filename=package://robot_properties_fingers/meshes/stl/pro/SIM__BL-F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 scale=1.0 1.0 1.0; visual mesh filename=package://robot_properties_fingers/meshes/stl/pro/SIM__BL-F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 scale=1.0 1.0 1.0
- link finger_tip_link_120: geometry collision mesh filename=package://robot_properties_fingers/meshes/stl/pro/SIM__BL-F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 scale=1.0 1.0 1.0; visual mesh filename=package://robot_properties_fingers/meshes/stl/pro/SIM__BL-F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 scale=1.0 1.0 1.0
- link finger_tip_link_240: geometry collision mesh filename=package://robot_properties_fingers/meshes/stl/pro/SIM__BL-F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 scale=1.0 1.0 1.0; visual mesh filename=package://robot_properties_fingers/meshes/stl/pro/SIM__BL-F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 scale=1.0 1.0 1.0
